File: Kicad_v2/01-power.kicad_sch (KiCad schematic)
At the start: 45 parts, among them IC2 BQ25630YBGR, J1 USB4105-GF-A-060, U11 RT6158HWSC, U2 TCR3UG33A_LF, U4 TPS61253F, U7 USBLC6-2SC6

Commit message: KiCad GPS en LoRa herschikt en gecombineerd
Parts:
- IC2: footprint BGA30C40P5X6_221X271X50 -> BQ25630YBGR:BGA30C40P5X6_221X271X50
- L2: footprint Inductor_SMD:L_0402_1005Metric -> MAKK2520H1R0M:MAKK2520H1R0M
- U1: renamed from U11; footprint BGA25_RT6158H_RIT -> RT6158AWSC:BGA25_RT6158H_RIT-M
Connections:
- net GPS_EN: now also U2.B1 (CTRL)
Other:
- moved on the sheet: C10, C11, C12, C13, C42, C43, L3, R12, R13, U2, U4

Commit message: PCB routing claude (deel 1)
Parts:
- J1: footprint Connector_USB:USB_C_Receptacle_GCT_USB4105-xx-A_16P_TopMnt_Horizontal -> USB-C:USB_C_Receptacle_GCT_USB4105-xx-A_16P_TopMnt_Horizontal
Changed lines of the file:
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@@
 			)
 		)
-		(property "Footprint" "Connector_USB:USB_C_Receptacle_GCT_USB4105-xx-A_16P_TopMnt_Horizontal"
+		(property "Footprint" "USB-C:USB_C_Receptacle_GCT_USB4105-xx-A_16P_TopMnt_Horizontal"
 			(at 57.658 73.66 0)
 			(hide yes)
@@
 		(in_pos_files yes)
 		(dnp no)
-		(property "Reference" "#PWR013"
+		(property "Reference" "#PWR036"
 			(at 180.34 85.09 0)
 			(hide yes)
@@
 			(project "Bikera PCB devboard"
 				(path "/81c195cb-438f-45ca-b649-b955fa3ba763/fe83c9ae-cf0a-47eb-9472-8f920f69f9b8"
-					(reference "#PWR013")
+					(reference "#PWR036")
 					(unit 1)
 				)
@@
 		(in_pos_files yes)
 		(dnp no)
-		(property "Reference" "#PWR017"
+		(property "Reference" "#PWR038"
 			(at 73.66 77.47 0)
 			(hide yes)
@@
 			(project "Bikera PCB devboard"
 				(path "/81c195cb-438f-45ca-b649-b955fa3ba763/fe83c9ae-cf0a-47eb-9472-8f920f69f9b8"
-					(reference "#PWR017")
+					(reference "#PWR038")
 					(unit 1)
 				)
@@
 		(in_pos_files yes)
 		(dnp no)
-		(property "Reference" "#PWR016"
+		(property "Reference" "#PWR037"
 			(at 73.66 30.48 0)
 			(hide yes)
@@
 			(project "Bikera PCB devboard"
 				(path "/81c195cb-438f-45ca-b649-b955fa3ba763/fe83c9ae-cf0a-47eb-9472-8f920f69f9b8"
-					(reference "#PWR016")
+					(reference "#PWR037")
 					(unit 1)
 				)
@@
 		(in_pos_files yes)
 		(dnp no)
-		(property "Reference" "#PWR018"
+		(property "Reference" "#PWR039"
 			(at 261.62 95.25 0)
 			(hide yes)
@@
 			(project "Bikera PCB devboard"
 				(path "/81c195cb-438f-45ca-b649-b955fa3ba763/fe83c9ae-cf0a-47eb-9472-8f920f69f9b8"
-					(reference "#PWR018")
+					(reference "#PWR039")
 					(unit 1)
 				)
@@
 		(in_pos_files yes)
 		(dnp no)
-		(property "Reference" "#PWR020"
+		(property "Reference" "#PWR040"
 			(at 194.31 149.86 0)
 			(hide yes)
@@
 			(project "Bikera PCB devboard"
 				(path "/81c195cb-438f-45ca-b649-b955fa3ba763/fe83c9ae-cf0a-47eb-9472-8f920f69f9b8"
-					(reference "#PWR020")
+					(reference "#PWR040")
 					(unit 1)
 				)

Commit message: Update laatste controle schema
Parts:
- removed R1, R2: 5.1K, Resistor_SMD:R_0603_1608Metric_Pad0.98x0.95mm_HandSolder, symbol Device:R
- added R29: 10 kΩ, Resistor_SMD:R_0603_1608Metric_Pad0.98x0.95mm_HandSolder, symbol Device:R
- U1: value RT6158HWSC -> RT6158AWSC
Connections:
- net CHRG_CE: now also R29.2
- net GND: now also R29.1
- net D-: now reaches U7.4 (I/O2)
- net D-: now also IC2.F3 (D-)
- net D+: now reaches U7.6 (I/O1)
- net D+: now also IC2.F2 (D+)
- no-connect marks 7 -> 3
Other:
- moved on the sheet: J1, R5, R6, U7
