File: Kicad_v2/02-mcu.kicad_sch (KiCad schematic)
At the start: 32 parts, among them IC1 DRV5032DULPGM, IC3 DRV5032DULPGM, J3 ST-LINK BTB, SW1 SW_Push, SW2 SW_Push, U3 STM32L431CCTx, U5 ATECC608B-SSHDA-T

Commit message: KiCad MCU schema gecontroleerd
Parts:
- removed C21: 22µF, Capacitor_SMD:C_0402_1005Metric, symbol Device:C_Small
- removed H1: TD-8120MG, Connector_JST:JST_PH_B3B-PH-K_1x03_P2.00mm_Vertical, symbol TD-8120MG:TD-8120MG
- removed J: B3B-ZR, B3B-ZR:B3B-ZR, symbol B3B-ZR:B3B-ZR
- added C21: 470µF, Capacitor_THT:CP_Radial_D8.0mm_P3.50mm, symbol Device:C_Polarized_Small
- added C40: 100nF, Capacitor_SMD:C_0603_1608Metric_Pad1.08x0.95mm_HandSolder, symbol Device:C_Small
- added C41: 4.7µF, Capacitor_SMD:C_0603_1608Metric_Pad1.08x0.95mm_HandSolder, symbol Device:C_Small
- added H4: TD-8120MG, Connector_JST:JST_PH_B3B-PH-K_1x03_P2.00mm_Vertical, symbol TD-8120MG:TD-8120MG
- added R26: 1K, Resistor_SMD:R_0603_1608Metric_Pad0.98x0.95mm_HandSolder, symbol Device:R
- C14, C15, C16, C17, C19, C20, C23, C24, C25, C26, C27: footprint Capacitor_SMD:C_0402_1005Metric -> Capacitor_SMD:C_0603_1608Metric_Pad1.08x0.95mm_HandSolder
- C18: value 100nF -> 10nF; footprint Capacitor_SMD:C_0402_1005Metric -> Capacitor_SMD:C_0603_1608Metric_Pad1.08x0.95mm_HandSolder
- C22: value 100nF -> 33nF; footprint Capacitor_SMD:C_0402_1005Metric -> Capacitor_SMD:C_0603_1608Metric_Pad1.08x0.95mm_HandSolder
- D1: footprint (none) -> LED_THT:LED_D5.0mm-3_Horizontal_O3.81mm_Z3.0mm
- FB1: footprint (none) -> Inductor_SMD:L_0603_1608Metric_Pad1.05x0.95mm_HandSolder
- R14: value 470Ω -> 160Ω; footprint Resistor_SMD:R_0402_1005Metric -> Resistor_SMD:R_0603_1608Metric_Pad0.98x0.95mm_HandSolder
- R15: value 330Ω -> 130Ω; footprint Resistor_SMD:R_0402_1005Metric -> Resistor_SMD:R_0603_1608Metric_Pad0.98x0.95mm_HandSolder
- R16: value 0.05 Ω, 2 W -> 0.1 Ω, 500mW; footprint (none) -> Resistor_SMD:R_1206_3216Metric_Pad1.30x1.75mm_HandSolder
- R17, R3, R4: footprint Resistor_SMD:R_0402_1005Metric -> Resistor_SMD:R_0603_1608Metric_Pad0.98x0.95mm_HandSolder
- SW1: value SW_Push -> SW_Reset; footprint (none) -> Button_Switch_THT:SW_PUSH_6mm
- SW2: value SW_Push -> SW_Boot; footprint (none) -> Button_Switch_THT:SW_PUSH_6mm
- U5: footprint ATECC608B-SSHDA-T:SOIC127P600X175-8N -> Package_DIP:DIP-8_W7.62mm_Socket
Connections:
- net +3V3: now also SW2.1, C41.1, C41.2; no longer R17.2
- net +5V: now also C21.2, H4.1 (VCC)
- net GND: now also R17.2, C21.1, C40.1
- net SERVO_PWM: now also H4.3 (SIG)
- net at R17.1: now also SW2.2, U3.44 (PH3); no longer SW2.1
- net at C17.2, C18.2, FB1.1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: now also C40.2
- net SERVO_ISENSE: no longer names the net of C22.2, R16.2
- net SERVO_ISENSE: now also H4.2 (GND), R26.1; no longer U3.18 (PB0)
- new net SERVO_RSENSE: R26.2, U3.18 (PB0)
Other:
- note removed: "rail sack? 470uF polarized"
- moved on the sheet: C14, C15, C16, C17, C18, C20, D1, J3, R14, R15, R16, R17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
