File: Kicad_v2/02-mcu.kicad_sch (KiCad schematic)
At the start: 34 parts, among them IC1 DRV5032DULPGM, IC3 DRV5032DULPGM, J3 ST-LINK BTB, SW1 SW_Reset, SW2 SW_Boot, U3 STM32L431CCTx, U5 ATECC608B-SSHDA-T

Commit message: KiCad GPS en LoRa herschikt en gecombineerd
Parts:
- J3: footprint 009159010603906 -> 009159010603906:009159010603906
Changed lines of the file:
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@@
 			)
 		)
-		(property "Footprint" "009159010603906"
+		(property "Footprint" "009159010603906:009159010603906"
 			(at 234.95 200.33 0)
 			(hide yes)

Commit message: PCB routing claude (deel 1)
Parts:
- IC1, IC3: footprint DRV5032DULPGM -> DRV5032DULPGM:DRV5032DULPGM
Changed lines of the file:
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@@
 		(in_pos_files yes)
 		(dnp no)
-		(property "Reference" "#PWR014"
+		(property "Reference" "#PWR042"
 			(at 25.4 13.97 0)
 			(hide yes)
@@
 			(project "Bikera PCB devboard"
 				(path "/81c195cb-438f-45ca-b649-b955fa3ba763/4ad3ced7-d468-45e1-aabd-eb3988119771"
-					(reference "#PWR014")
+					(reference "#PWR042")
 					(unit 1)
 				)
@@
 		(in_pos_files yes)
 		(dnp no)
-		(property "Reference" "#PWR015"
+		(property "Reference" "#PWR041"
 			(at 19.05 24.13 0)
 			(hide yes)
@@
 			(project "Bikera PCB devboard"
 				(path "/81c195cb-438f-45ca-b649-b955fa3ba763/4ad3ced7-d468-45e1-aabd-eb3988119771"
-					(reference "#PWR015")
+					(reference "#PWR041")
 					(unit 1)
 				)
@@
 			)
 		)
-		(property "Footprint" "DRV5032DULPGM"
+		(property "Footprint" "DRV5032DULPGM:DRV5032DULPGM"
 			(at 44.45 47.32 0)
 			(hide yes)
@@
 			)
 		)
-		(property "Footprint" "DRV5032DULPGM"
+		(property "Footprint" "DRV5032DULPGM:DRV5032DULPGM"
 			(at 44.45 15.57 0)
 			(hide yes)
